File: Digijet.kicad_sch (KiCad schematic)
At the start: 65 parts, among them J1 Conn_01x25, Q1 BC337, Q2 BC618, Q3 BC618, Q4 BD238, U1 LM2901, U2 74LS373, U3 74LS00, U4 2764, U5 8039, U6 ADC0809, U7 TA7900S, Y1 Crystal_GND3

Commit message: alle tht teile
Parts:
- added C19: C, Capacitor_THT:C_Rect_L24.0mm_W7.0mm_P22.50mm_MKT, symbol Device:C
- added C20, C31: C, Capacitor_THT:C_Rect_L7.0mm_W3.5mm_P5.00mm, symbol Device:C
- added C21, C22, C23, C24, C25, C26, C27, C28, C29, C30: C, Capacitor_THT:C_Disc_D4.3mm_W1.9mm_P5.00mm, symbol Device:C
- added D8, D9: D, Diode_THT:D_A-405_P12.70mm_Horizontal, symbol Device:D
- added Q5: Q_NPN_Darlington_BCE, Package_TO_SOT_THT:TO-220-3_Vertical, symbol Transistor_BJT:Q_NPN_Darlington_BEC
- added R27, R28, R29, R30, R31, R32, R33, R34, R35, R36, R37, R38, R39, R40, R41, R42, R47, R49, R51, R52, R53, R54, R55, R56, R57: R, Resistor_THT:R_Axial_DIN0207_L6.3mm_D2.5mm_P10.16mm_Horizontal, symbol Device:R
- added R43: 10R 5%, Resistor_THT:R_Axial_DIN0414_L11.9mm_D4.5mm_P25.40mm_Horizontal, symbol Device:R
- added R44, R46, R48, R50: R, Resistor_THT:R_Axial_DIN0207_L6.3mm_D2.5mm_P15.24mm_Horizontal, symbol Device:R
- added R45: Power, Resistor_THT:R_Axial_DIN0516_L15.5mm_D5.0mm_P30.48mm_Horizontal, symbol Device:R
- added R58: 0, Resistor_THT:R_Axial_DIN0207_L6.3mm_D2.5mm_P7.62mm_Horizontal, symbol Device:R
- added R59: Power, Resistor_THT:R_Axial_DIN0309_L9.0mm_D3.2mm_P15.24mm_Horizontal, symbol Device:R
- C10, C17, C3, C4, C5, C6, C7, C8: footprint Capacitor_THT:C_Rect_L7.0mm_W2.0mm_P5.00mm -> Capacitor_THT:C_Rect_L7.0mm_W3.5mm_P5.00mm
- C11, C12, C18, C9: footprint Capacitor_THT:CP_Radial_Tantal_D4.5mm_P5.00mm -> Capacitor_THT:C_Disc_D4.3mm_W1.9mm_P5.00mm; symbol Device:C_Polarized -> Device:C
- C13: footprint Capacitor_THT:C_Rect_L7.0mm_W4.5mm_P5.00mm -> Capacitor_THT:C_Rect_L7.0mm_W3.5mm_P5.00mm
- J1: footprint (none) -> Connector_VW:ZIP-25
Connections:
- net ALE: now also U2.11 (LE)
- net GND: now also D6.2 (A), J1.10 (Pin_10), J1.16 (Pin_16), J1.17 (Pin_17), J1.18 (Pin_18), J1.22 (Pin_22), J1.3 (Pin_3), J1.6 (Pin_6), J1.7 (Pin_7), J1.9 (Pin_9), Q1.3 (E), R15.1, R16.1, C20.2, C21.2, C22.1, C24.2, C26.2, C28.2, C29.2, C30.2, C31.2, D9.2 (A), R29.2, R44.2, R46.2, R47.2, R48.2, R49.2, R50.2, R51.2, R52.1, R55.1, R56.1, R58.1
- net P2.5: now also R38.2
- net P2.6: now also R37.2
- net RD: now also U6.22 (ALE)
- net VCC: now also R28.2, R30.2, R31.2, R34.2, R43.2
- net at Q1.1 (C): now also R3.2, U3.10
- net at Q1.2 (B): now also R2.2, R55.2
- net at C17.1, D3.1 (K), Q2.2 (B)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: now also D7.1 (K)
- net C4: now reaches R12.1
- net C4: now also J1.4 (Pin_4), R35.2
- net THROTTLE: now reaches C3.1, D1.2 (A), R12.2, U5.1 (T0)
- net at R22.1: now also D5.2 (A), Q3.1 (C)
- net at R23.2: now also U7.6 (ADJ), R44.1
- net AIR_TEMP: now reaches U6.1 (IN3)
- net AIR_TEMP: now also C31.1, R33.2
- net AIR_AMOUNT: now reaches C5.1, U6.26 (IN0)
- net AIR_AMOUNT: now also R27.2
- net IGNITION: now reaches U6.27 (IN1)
- net IGNITION: now also C20.1, R52.2, R54.1
- net WATER_TEMP: now reaches C8.1, U6.28 (IN2)
- net WATER_TEMP: now also R32.2
- net at U1.14: now also R17.2, C23.2, R30.1
- net at R18.2, U1.8 (-): now also R15.2, C22.2
- net at U1.9 (+): now also R16.2, R17.1, C21.1
- net C21: now reaches R26.1
- net C21: now also J1.21 (Pin_21)
- net at C9.1, R6.1, R7.1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: now also R35.1, R39.2, R40.2, R41.2
- net C1: now reaches J1.1 (Pin_1)
- net C1: now also R18.1, C24.1
- net C11: now reaches J1.11 (Pin_11)
- net C11: now also J1.12 (Pin_12), J1.23 (Pin_23), J1.24 (Pin_24), C28.1, Q5.2 (E), R45.1
- net C13: now reaches J1.13 (Pin_13)
- net C13: now also D8.2 (A), R54.2
- net C14: now reaches J1.14 (Pin_14)
- net C14: now also R33.1, R34.1
- net C15: now reaches J1.15 (Pin_15)
- net C15: now also R27.1, R29.1
- net C19: now reaches J1.19 (Pin_19)
- net C19: now also R43.1
- net C2: now reaches J1.2 (Pin_2)
- net C2: now also R31.1, R32.1
- net C20: now reaches J1.20 (Pin_20)
- net C20: now also Q2.1 (C), C29.1, R56.2
- net C25: now reaches J1.25 (Pin_25)
- net C25: now also C19.1, C30.1, D9.1 (K), Q5.3 (C), R57.1
- net C5: now reaches J1.5 (Pin_5)
- net C5: now also R36.2
- net C8: now reaches J1.8 (Pin_8)
- net at D5.1 (K): now also Q5.1 (B), R57.2
- net LAMBDA: now reaches U1.4 (-), U1.6 (-)
- net LAMBDA: now also C25.2, C26.1, C27.1, R36.1, R42.2
- net at U1.7 (+): now also C25.1, R37.1, R39.1, R46.1, R47.1
- net at U1.5 (+): now also C27.2, R38.1, R40.1, R48.1, R49.1
- net P1.1: no longer names the net of U5.28 (P1.1)
- net P1.2: no longer names the net of U5.29 (P1.2)
- net P1.7: no longer names the net of U5.34 (P1.7)
- net P2.4: no longer names the net of U5.35 (P2.4)
- net P2.7: no longer names the net of U5.38 (P2.7)
- new net: C23.1, R28.1
- new net: R41.1, R42.1, R50.1, R51.1
- new net: D8.1 (K), R59.2
- new net: C19.2, R45.2
- no-connect marks 1 -> 9
Other:
- moved on the sheet: C15, D2, D5, D6, D7, J1, Q1, Q3, R15, R16, R17, R2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

Commit message: smd
Parts:
- added C32, C33, C34, C35, C36, C37, C38, C39, C40, C41, C42, C43, C44, C45: C, Capacitor_SMD:C_1206_3216Metric, symbol Device:C
- added H1: MountingHole, MountingHole:MountingHole_2.5mm, symbol Mechanical:MountingHole
- C1, C2: value C -> 22P
- RN1: value R_Network06_Split -> 5X-1-472
- Y1: value Crystal_GND3 -> 7.372800
Connections:
- net C1: now also C42.2
- net C11: now also C35.2
- net C13: now also C34.2
- net C14: now also C44.2
- net C15: now also C45.2
- net C19: now also C41.2
- net C2: now also C43.2
- net C20: now also C39.2
- net C21: now also C38.2
- net C25: now also C33.2
- net C5: now also C37.2
- net C8: now also C36.2
- net GND: now also C40.2
- net VCC: now also C9.1, R35.1, R39.2, R40.2, R41.2, R6.1, R7.1, U1.3 (V+)
- net at R20.2: now also C13.1, U7.8 (TC)
- net at C16.1, C18.1, Q4.1 (E)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: now also R53.2, R59.1
- net at C23.1, R28.1: now also D2.2 (A), R2.1
- net at R53.1: now also C21.1, R16.2, R17.1, U1.9 (+)
- net at R58.2: now also C32.2
- net A11: no longer names the net of R14.1, U4.23 (A11)
- new net: C32.1, C33.1, C34.1, C35.1, C36.1, C37.1, C38.1, C39.1, C40.1, C41.1, C42.1, C43.1, C44.1, C45.1
Other:
- moved on the sheet: C1, C10, C15, C2, C3, C4, C7, C9, D1, D2, Q1, R1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
