File: Digijet/Digijet.kicad_sch (KiCad schematic)
At the start: 129 parts, among them J1 Conn_01x25, Q1 BC337, Q2 BC618, Q3 BC618, Q4 BD238, Q5 Q_NPN_Darlington_BCE, U1 LM2901, U2 74LS373, U3 74LS00, U4 2764, U5 8039, U6 ADC0809, U7 TA7900S, Y1 7.372800

Commit message: widerstand werte
Parts:
- removed R56: R, Resistor_THT:R_Axial_DIN0207_L6.3mm_D2.5mm_P10.16mm_Horizontal, symbol Device:R
- added D10: ZPDxx, Diode_THT:D_DO-35_SOD27_P10.16mm_Horizontal, symbol Diode:ZPDxx
- added Q6: BC337, Package_TO_SOT_THT:TO-92_Inline_Wide, symbol Transistor_BJT:BC337
- added R60, R61: R, Resistor_THT:R_Axial_DIN0207_L6.3mm_D2.5mm_P10.16mm_Horizontal, symbol Device:R
- added R62: 0, Resistor_THT:R_Axial_DIN0207_L6.3mm_D2.5mm_P7.62mm_Horizontal, symbol Device:R
- C10, C17, C20, C3, C31, C4, C5, C6, C7, C8: value C -> 0.22 63-B
- C11: value C_Polarized -> 332K
- C12, C18, C9: value C_Polarized -> 104K
- C13: value C -> 0.68 63
- C15: value C_Polarized -> 63V 47uF
- C16: value C_Polarized -> 40V 220uF
- C19: value C -> 1.5uF 100-A
- C21, C22, C29: value C -> 103K
- C23: value C -> 332K
- C24: value C -> 102K
- C26, C30: value C -> 104K
- C27: value C -> 223K
- C28: value C -> 473K
- C32, C33, C34, C35, C36, C37, C38, C39, C40, C41, C42, C43, C44, C45: value C -> 28nF
- Q5: value Q_NPN_Darlington_BCE -> TE2443
- R1: value R -> 1k 1%
- R10, R11, R13, R6, R7: value R -> 5.11k 1%
- R12, R32, R33: value R -> 14.2k 1% 50ppm
- R15, R19, R20, R25, R27, R30, R36, R39, R40, R41: value R -> 10k 1%
- R16: value R -> 4.75k 1% 50ppm
- R17: value R -> 100k 1%
- R18: value R -> 22.1k 1% 50ppm
- R2: value R -> 5.62k 1% 50ppm
- R21: value R -> 15k 1% 50ppm
- R22: value R -> 4.7k 2%
- R23: value R -> 1.6M
- R26, R28: value R -> 3.32k 1%
- R29: value R -> 140 1%
- R3: value R -> 2k 1%
- R31, R34: value R -> 4.26k 1%
- R35: value R -> 475 1% 50ppm
- R37: value R -> 475k 1% 50ppm
- R38: value R -> 2.13k 1%
- R4: value R -> 1.5k 1%
- R42: value R -> 39.2k 1% 50ppm
- R45: value Power -> 23
- R46: value R -> 16.1k 1%
- R47: value R -> 1.1k 1%
- R48: value R -> 12.1k 1%
- R49: value R -> 1.33k 1% 50ppm
- R5, R54: value R -> 20k 1% 50ppm
- R50: value R -> 14.7k 1%
- R51: value R -> 1.21k 1%
- R52: value R -> 4.63k 1%
- R53: value R -> 47.6k 1%
- R55: value R -> 3.92k 1%
- R57: value R -> 750 1%
- R59: value Power -> 0.17 5%
- R8, R9: value R -> 825 1%
Connections:
- net C20: now also D10.1 (K)
- net C8: now also R61.2
- net GND: now also D10.2 (A), Q6.3 (E), R60.1
- net P1.3: now also Q6.2 (B)
- net at R14.1, U4.23 (A11): now also R62.2
- net P2.3 renamed A11
- net A11: now also R62.1
- new net: Q6.1 (C), R60.2, R61.1
- no-connect marks 9 -> 12
Other:
- moved on the sheet: C1, C11, C12, C13, C14, C16, C17, C18, C19, C2, C20, C21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
